Commit message: term

File: src/twolink_gazebo/urdf/twolinkbot.urdf.xacro (robot description, xacro)
@@ -1,5 +1,5 @@
 <?xml version="1.0"?>
 <robot name="twolinkbot" xmlns:xacro="http://ros.org/wiki/xacro">
-    <xacro:include filename="macros.xacro"/>
+  <xacro:include filename="macros.xacro"/>
   <link name="world">
   </link>
@@ -10,5 +10,5 @@
   <link name="base_link">
     <visual>
-        <origin xyz="0 0 0"/>
+        <origin xyz="0.045 0.05 0"/>
         <geometry>
           <mesh
@@ -16,9 +16,9 @@
         </geometry>
         <material name="grey">
-            <color rgba="0.5 0.5 0.5 1.0"/> <!-- 회색 -->
+            <color rgba="0.5 0.5 0.5 1.0"/>
         </material>
     </visual>
     <collision>
-        <origin xyz="0 0 0"/>
+        <origin xyz="0.045 0.05 0"/>
         <geometry>
           <mesh
@@ -30,27 +30,16 @@
     </xacro:inertial_cylinder>
   </link>
-  <joint name="joint1" type="continuous">
-    <parent link="base_link"/>
-    <child link="link1"/>
-    <origin xyz="-0.045 -0.05 0.09435"/>
-    <axis xyz="0 0 1"/>
+  <!--START OF YOUR CODE-->
+  <joint name="joint1" type="">
+    <!--END OF YOUR CODE-->
   </joint>
   <link name="link1">
     <visual>
-        <origin xyz="0 0 0"/>
-        <geometry>
-          <mesh
-          filename="file://$(find twolink_gazebo)/meshes/link1.stl" />
-        </geometry>
-        <material name="grey">
-            <color rgba="0.5 0.5 0.5 1.0"/> <!-- 회색 -->
-        </material>
+      <!--START OF YOUR CODE-->
+      <!--END OF YOUR CODE-->
     </visual>
     <collision>
-        <origin xyz="0 0 0"/>
-        <geometry>
-          <mesh
-          filename="file://$(find twolink_gazebo)/meshes/link1.stl" />
-        </geometry>
+      <!--START OF YOUR CODE-->
+      <!--END OF YOUR CODE-->
     </collision>
     <xacro:inertial_box mass="0.5" x="0.2" y="0.057" z="0.057">
@@ -58,27 +47,16 @@
     </xacro:inertial_box>
   </link>
-  <joint name="joint2" type="continuous">
-    <parent link="link1"/>
-    <child link="link2"/>
-    <origin xyz="-0.143 0 0.09365"/>
-    <axis xyz="0 0 1"/>
+  <!--START OF YOUR CODE-->
+  <joint name="joint2" type="">
+    <!--END OF YOUR CODE-->
   </joint>
   <link name="link2">
     <visual>
-        <origin xyz="0 0 0"/>
-        <geometry>
-          <mesh
-          filename="file://$(find twolink_gazebo)/meshes/link2.stl" />
-        </geometry>
-        <material name="grey">
-            <color rgba="0.5 0.5 0.5 1.0"/> <!-- 회색 -->
-        </material>
+      <!--START OF YOUR CODE-->
+      <!--END OF YOUR CODE-->
     </visual>
     <collision>
-        <origin xyz="0 0 0"/>
-        <geometry>
-          <mesh
-          filename="file://$(find twolink_gazebo)/meshes/link2.stl" />
-        </geometry>
+      <!--START OF YOUR CODE-->
+      <!--END OF YOUR CODE-->
     </collision>
     <xacro:inertial_box mass="0.2" x="0.15" y="0.048" z="0.006">
@@ -99,5 +77,5 @@
         </geometry>
         <material name="grey">
-            <color rgba="0.5 0.5 0.5 1.0"/> <!-- 회색 -->
+            <color rgba="0.5 0.5 0.5 1.0"/>
         </material>
     </visual>
@@ -113,9 +91,9 @@
     <parent link="d435_holder"/>
     <child link="d435"/>
-    <origin xyz="0 0 0.006"/>
+    <origin xyz="0 0 0.018" rpy="0 0 3.14159"/>
   </joint>
   <link name="d435">
     <visual>
-        <origin xyz="0 0 0" rpy="0 0 3.14159"/>
+        <origin xyz="0 0 -0.012" rpy="0 0 0"/>
         <geometry>
           <mesh
@@ -127,5 +105,5 @@
     </visual>
     <collision>
-        <origin xyz="0 0 0" rpy="0 0 3.14159"/>
+        <origin xyz="0 0 -0.012" rpy="0 0 0"/>
         <geometry>
           <mesh

Commit message: Add files via upload

File: src/twolink_gazebo/urdf/twolinkbot.urdf.xacro (robot description, xacro)
@@ -10,5 +10,5 @@
   <link name="base_link">
     <visual>
-        <origin xyz="0.045 0.05 0"/>
+        <origin xyz="-0.045 -0.05 0"/>
         <geometry>
           <mesh
@@ -20,5 +20,5 @@
     </visual>
     <collision>
-        <origin xyz="0.045 0.05 0"/>
+        <origin xyz="-0.045 -0.05 0"/>
         <geometry>
           <mesh
@@ -31,5 +31,9 @@
   </link>
   <!--START OF YOUR CODE-->
-  <joint name="joint1" type="">
+  <joint name="joint1" type="continuous">
+    <parent link="base_link"/>
+    <child link="link1"/>
+    <origin xyz="0 0 0.09435" rpy="0 0 0"/>
+    <axis xyz="0.0 0.0 1.0"/>
     <!--END OF YOUR CODE-->
   </joint>
@@ -37,16 +41,31 @@
     <visual>
       <!--START OF YOUR CODE-->
+      <origin xyz="0.0 0.0 0.0"/>
+      <geometry>
+        <mesh filename="file://$(find twolink_gazebo)/meshes/link1.stl" />
+      </geometry>
+      <material name="grey">
+          <color rgba="0.5 0.5 0.5 1.0"/>
+      </material>
       <!--END OF YOUR CODE-->
     </visual>
     <collision>
       <!--START OF YOUR CODE-->
+      <origin xyz="0.0 0.0 0.0"/>
+      <geometry>
+        <mesh filename="file://$(find twolink_gazebo)/meshes/link1.stl" />
+      </geometry>
       <!--END OF YOUR CODE-->
     </collision>
     <xacro:inertial_box mass="0.5" x="0.2" y="0.057" z="0.057">
             <origin xyz="-0.0715 0 0.03"/>
-    </xacro:inertial_box>
+    </xacro:inertial_box>link2
   </link>
   <!--START OF YOUR CODE-->
-  <joint name="joint2" type="">
+  <joint name="joint2" type="continuous">
+    <parent link="link1"/>
+    <child link="link2"/>
+    <origin xyz="0.143 0 0.09365" rpy="0 0 0"/>
+    <axis xyz="0.0 0.0 1.0"/>
     <!--END OF YOUR CODE-->
   </joint>
@@ -54,8 +73,19 @@
     <visual>
       <!--START OF YOUR CODE-->
+      <origin xyz="0.0 0.0 0.0"/>
+      <geometry>
+        <mesh filename="file://$(find twolink_gazebo)/meshes/link2.stl" />
+      </geometry>
+      <material name="grey">
+          <color rgba="0.5 0.5 0.5 1.0"/>
+      </material>
       <!--END OF YOUR CODE-->
     </visual>
     <collision>
       <!--START OF YOUR CODE-->
+      <origin xyz="0.0 0.0 0.0"/>
+      <geometry>
+        <mesh filename="file://$(find twolink_gazebo)/meshes/link2.stl" />
+      </geometry>
       <!--END OF YOUR CODE-->
     </collision>
@@ -67,9 +97,9 @@
     <parent link="link2"/>
     <child link="d435_holder"/>
-    <origin xyz="-0.102 0 0.021"/>
+    <origin xyz="0.102 0 0.021"/>
   </joint>
   <link name="d435_holder">
     <visual>
-        <origin xyz="0 0 0" rpy="0 0 3.14159"/>
+        <origin xyz="0 0 0" rpy="0 0 0"/>
         <geometry>
           <mesh
@@ -81,5 +111,5 @@
     </visual>
     <collision>
-        <origin xyz="0 0 0" rpy="0 0 3.14159"/>
+        <origin xyz="0 0 0" rpy="0 0 0"/>
         <geometry>
           <mesh
@@ -91,5 +121,5 @@
     <parent link="d435_holder"/>
     <child link="d435"/>
-    <origin xyz="0 0 0.018" rpy="0 0 3.14159"/>
+    <origin xyz="0 0 0.018" rpy="0 0 0"/>
   </joint>
   <link name="d435">

Commit message: 2025-2

File: src/twolink_gazebo/urdf/twolinkbot.urdf.xacro (robot description, xacro)
@@ -30,10 +30,6 @@
     </xacro:inertial_cylinder>
   </link>
-  <!--START OF YOUR CODE-->
-  <joint name="joint1" type="continuous">
-    <parent link="base_link"/>
-    <child link="link1"/>
-    <origin xyz="0 0 0.09435" rpy="0 0 0"/>
-    <axis xyz="0.0 0.0 1.0"/>
+    <!--START OF YOUR CODE-->
+    <joint name="joint1" type="">
     <!--END OF YOUR CODE-->
   </joint>
@@ -41,19 +37,8 @@
     <visual>
       <!--START OF YOUR CODE-->
-      <origin xyz="0.0 0.0 0.0"/>
-      <geometry>
-        <mesh filename="file://$(find twolink_gazebo)/meshes/link1.stl" />
-      </geometry>
-      <material name="grey">
-          <color rgba="0.5 0.5 0.5 1.0"/>
-      </material>
       <!--END OF YOUR CODE-->
     </visual>
     <collision>
       <!--START OF YOUR CODE-->
-      <origin xyz="0.0 0.0 0.0"/>
-      <geometry>
-        <mesh filename="file://$(find twolink_gazebo)/meshes/link1.stl" />
-      </geometry>
       <!--END OF YOUR CODE-->
     </collision>
@@ -62,10 +47,6 @@
     </xacro:inertial_box>link2
   </link>
-  <!--START OF YOUR CODE-->
-  <joint name="joint2" type="continuous">
-    <parent link="link1"/>
-    <child link="link2"/>
-    <origin xyz="0.143 0 0.09365" rpy="0 0 0"/>
-    <axis xyz="0.0 0.0 1.0"/>
+    <!--START OF YOUR CODE-->
+    <joint name="joint2" type="">
     <!--END OF YOUR CODE-->
   </joint>
@@ -73,19 +54,8 @@
     <visual>
       <!--START OF YOUR CODE-->
-      <origin xyz="0.0 0.0 0.0"/>
-      <geometry>
-        <mesh filename="file://$(find twolink_gazebo)/meshes/link2.stl" />
-      </geometry>
-      <material name="grey">
-          <color rgba="0.5 0.5 0.5 1.0"/>
-      </material>
       <!--END OF YOUR CODE-->
     </visual>
     <collision>
       <!--START OF YOUR CODE-->
-      <origin xyz="0.0 0.0 0.0"/>
-      <geometry>
-        <mesh filename="file://$(find twolink_gazebo)/meshes/link2.stl" />
-      </geometry>
       <!--END OF YOUR CODE-->
     </collision>
